Commit message: Fix joint type to revolute and add joint limits

File: moveit_6dof_arm/config/urdf_6dof_arm.ros2_control.xacro (robot description, xacro)
@@ -2,5 +2,5 @@
 <robot xmlns:xacro="http://www.ros.org/wiki/xacro">
     <xacro:macro name="urdf_6dof_arm_ros2_control" params="name initial_positions_file">
-        <xacro:property name="initial_positions" value="${load_yaml(initial_positions_file)['initial_positions']}"/>
+        <xacro:property name="initial_positions" value="${xacro.load_yaml(initial_positions_file)['initial_positions']}"/>
         <ros2_control name="${name}" type="system">
             <hardware>
@@ -8,52 +8,74 @@
                 <plugin>mock_components/GenericSystem</plugin>
             </hardware>
-            <joint name="Joint_1">
+            <joint name="Joint_1" type="revolute">
                 <command_interface name="position"/>
                 <state_interface name="position">
                   <param name="initial_value">${initial_positions['Joint_1']}</param>
                 </state_interface>
-                <state_interface name="velocity"/>
+                <state_interface name="velocity">
+                  <param name="initial_value">0.0</param>
+                </state_interface>
+                <limit lower="-3.14" upper="3.14" effort="2.94" velocity="4.5" />
             </joint>
-            <joint name="Joint_2">
+            <joint name="Joint_2" type="revolute">
                 <command_interface name="position"/>
                 <state_interface name="position">
                   <param name="initial_value">${initial_positions['Joint_2']}</param>
                 </state_interface>
-                <state_interface name="velocity"/>
+                <state_interface name="velocity">
+                  <param name="initial_value">0.0</param>
+                </state_interface>
+                <limit lower="-1.57" upper="1.57" effort="2.94" velocity="4.5" />
             </joint>
-            <joint name="Joint_3">
+            <joint name="Joint_3" type="revolute">
                 <command_interface name="position"/>
                 <state_interface name="position">
                   <param name="initial_value">${initial_positions['Joint_3']}</param>
                 </state_interface>
-                <state_interface name="velocity"/>
+                <state_interface name="velocity">
+                  <param name="initial_value">0.0</param>
+                </state_interface>
+                <limit lower="-1.57" upper="1.57" effort="2.94" velocity="4.5" />
             </joint>
-            <joint name="Joint_4">
+            <joint name="Joint_4" type="revolute">
                 <command_interface name="position"/>
                 <state_interface name="position">
                   <param name="initial_value">${initial_positions['Joint_4']}</param>
                 </state_interface>
-                <state_interface name="velocity"/>
+                <state_interface name="velocity">
+                  <param name="initial_value">0.0</param>
+                </state_interface>
+                <limit lower="-3.14" upper="3.14" effort="2.94" velocity="4.5" />
             </joint>
-            <joint name="Joint_5">
+            <joint name="Joint_5" type="revolute">
                 <command_interface name="position"/>
                 <state_interface name="position">
                   <param name="initial_value">${initial_positions['Joint_5']}</param>
                 </state_interface>
-                <state_interface name="velocity"/>
+                <state_interface name="velocity">
+                  <param name="initial_value">0.0</param>
+                </state_interface>
+                <limit lower="-1" upper="1.57" effort="2.94" velocity="4.5" />
             </joint>
-            <joint name="Joint_6">
+            <joint name="Joint_6" type="revolute">
                 <command_interface name="position"/>
                 <state_interface name="position">
                   <param name="initial_value">${initial_positions['Joint_6']}</param>
                 </state_interface>
-                <state_interface name="velocity"/>
+                <state_interface name="velocity">
+                  <param name="initial_value">0.0</param>
+                </state_interface>
+                <origin rpy="${pi/2} 0 0" />
+                <limit lower="-1.57" upper="3.14" effort="2.94" velocity="4.5" />
             </joint>
-            <joint name="Joint_Gripper">
+            <joint name="Joint_Gripper" type="revolute">
                 <command_interface name="position"/>
                 <state_interface name="position">
                   <param name="initial_value">${initial_positions['Joint_Gripper']}</param>
                 </state_interface>
-                <state_interface name="velocity"/>
+                <state_interface name="velocity">
+                  <param name="initial_value">0.0</param>
+                </state_interface>
+                <limit lower="-0.35" upper="0.6" effort="2.94" velocity="4.5" />
             </joint>
         </ros2_control>

File: urdf_6dof_arm/urdf/urdf_6dof_arm.urdf (robot description, URDF)
Before this commit: robot urdf_6dof_arm, 9 links, 8 joints
Joints:
- joint Joint_1: limit (none) -> lower=-3.14 upper=3.14 effort=2.94 velocity=4.5; type continuous -> revolute
- joint Joint_2: limit (none) -> lower=-1.57 upper=1.57 effort=2.94 velocity=4.5; type continuous -> revolute
- joint Joint_3: limit (none) -> lower=-1.57 upper=1.57 effort=2.94 velocity=4.5; type continuous -> revolute
- joint Joint_4: limit (none) -> lower=-3.14 upper=3.14 effort=2.94 velocity=4.5; type continuous -> revolute
- joint Joint_5: limit (none) -> lower=-1.46 upper=1.57 effort=2.94 velocity=4.5; type continuous -> revolute
- joint Joint_6: limit (none) -> lower=-1.57 upper=1.57 effort=2.94 velocity=4.5; origin xyz=0.0576950428676977 0 -0.00754999999999195 rpy=0 0 0 -> xyz=0.0576950428676977 0 -0.00754999999999195 rpy=${pi/2} 0 0; type continuous -> revolute
- joint Joint_Gripper: limit (none) -> lower=-0.35 upper=0.6 effort=2.94 velocity=4.5; type continuous -> revolute
