Commit message: Add a EE Gripper Link to urdf

File: arm_description/urdf/arm_description.urdf (robot description, URDF)
Before this commit: robot arm_description, 9 links, 8 joints
Links:
- added link EE_Gripper_Link, mass 0.0
Joints:
- added joint Joint_EE_Gripper: type fixed, parent Link_6, child EE_Gripper_Link, origin xyz=0.05 0 0 rpy=0 0 0

Commit message: Add EE_Gripper_Link as a virtual extension of Link_6 in urdf and srdf, update rviz default setup

File: arm_description/urdf/arm_description.urdf (robot description, URDF)
Before this commit: robot arm_description, 10 links, 9 joints
Joints:
- removed joint Joint_EE_Gripper
- added joint EE_Gripper_Joint: type fixed, parent Link_6, child EE_Gripper_Link, origin xyz=0.05 0 0 rpy=0 0 0
